File: hardware/blue-lighting.kicad_sch (KiCad schematic)
At the start: 0 parts

Commit message: Basic Decoupling, USB-C, and Reset Circuitry added
Parts:
- added 5.1K: R, symbol Device:R
- added C1, C10, C11, C13, C14, C19, C2, C3, C4, C5, C6, C7, C8, C9: 100nF, symbol Device:C
- added C12, C15: 1μF, symbol Device:C
- added C16, C17: 2.2μF, symbol Device:C
- added C18: 10μF, symbol Device:C
- added FB1: FerriteBead, symbol Device:FerriteBead
- added J1: USB_C_Receptacle_USB2.0_14P, symbol Connector:USB_C_Receptacle_USB2.0_14P
- added R1: 5.1K, symbol Device:R
- added SW1: CK_KMS2xxG, Button_Switch_SMD:SW_SPST_CK_KMS2xxGP, symbol Switch:CK_KMS2xxG
- added U1: STM32F767ZITx, Package_QFP:LQFP-144_20x20mm_P0.5mm, symbol MCU_ST_STM32F7:STM32F767ZITx
- added U2: NCP1117-1.5_SOT223, Package_TO_SOT_SMD:SOT-223-3_TabPin2, symbol Regulator_Linear:NCP1117-1.5_SOT223
Connections:
- new net: J1.A4 (VBUS), J1.A9 (VBUS), J1.B4 (VBUS), J1.B9 (VBUS), U2.3 (VI)
- new net: J1.A5 (CC1), R1.1
- new net: 5.1K.2, J1.B5 (CC2)
- new net: C17.1, U1.106 (VCAP_2)
- new net: C13.1, FB1.2
- new net: C12.1, C13.2
- new net: C14.2, C15.1
- new net: C16.1, U1.71 (VCAP_1)
- new net +3.3V: C1.1, C10.1, C11.1, C14.1, C18.1, C2.1, C3.1, C4.1, C5.1, C6.1, C7.1, C8.1, C9.1, FB1.1, U1.108 (VDD), U1.121 (VDDSDMMC), U1.131 (VDD), U1.143 (PDR_ON), U1.144 (VDD), U1.17 (VDD), U1.30 (VDD), U1.32 (VREF+), U1.33 (VDDA), U1.39 (VDD), U1.52 (VDD), U1.6 (VBAT), U1.62 (VDD), U1.72 (VDD), U1.84 (VDD), U1.95 (VDDUSB)
- new net GND: 5.1K.1, C1.2, C10.2, C11.2, C12.2, C15.2, C16.2, C17.2, C18.2, C19.2, C2.2, C3.2, C4.2, C5.2, C6.2, C7.2, C8.2, C9.2, J1.A1 (GND), J1.A12 (GND), J1.B1 (GND), J1.B12 (GND), J1.S1 (SHIELD), R1.2, SW1.1, U1.107 (VSS), U1.120 (VSS), U1.130 (VSS), U1.138 (BOOT0), U1.16 (VSS), U1.31 (VSSA), U1.38 (VSS), U1.51 (VSS), U1.61 (VSS), U1.83 (VSS), U1.94 (VSS), U2.1 (GND)
- new net NRST: U1.25 (NRST)
- new net NSRT: C19.1, SW1.2
- new net USB_D+: J1.A6 (D+), J1.B6 (D+)
- new net USB_D-: J1.A7 (D-), J1.B7 (D-)
Other:
- note added: "Capacitors for VDD and VBAT"
- note added: "Reset Button Circuit"
- note added: "VDDA"
- note added: "VREF+"
