File: hardware/blue-lightning.kicad_sch (KiCad schematic)
At the start: 28 parts, among them J1 USB_C_Receptacle_USB2.0_14P, SW1 CK_KMS2xxG, U1 STM32F767ZITx, U2 NCP1117-1.5_SOT223

Commit message: fixed mispellings and.gitgnore caches removed in hardware/
Parts:
- removed C20, C21: 10μF, symbol Device:C
Connections:
- net +3.3V: no longer U2.2 (VO)
- net PA11 renamed USB_D-
- net USB_D-: no longer U1.103 (PA11)
- net PA12 renamed USB_D+
- net USB_D+: no longer U1.104 (PA12)
- net VBUS: no longer names the net of J1.A4 (VBUS), J1.A9 (VBUS), J1.B4 (VBUS), J1.B9 (VBUS), U2.3 (VI)
Other:
- note removed: "USB OTG FS"
- moved on the sheet: U2
